File: Hardware/Simple/kicad/simple002.kicad_pcb (KiCad board)
At the start: 2 copper layers, 54.3 x 81.3 mm, 35 parts

Commit message: contd
Parts:
- added C1: 0.1uF, simple002:C2.5-3, F.Cu at (100.9, 113.4)
- added C2: 0.1uF, simple002:C2.5-3, F.Cu at (100.9, 117.6)
- added C3: 10uF, simple002:E2,5-5, F.Cu at (107.0, 114.4)
- added C4: 10uF, simple002:E2,5-5, F.Cu at (107.0, 120.7)
- added C5: 0.1uF, simple002:C2.5-3, F.Cu at (100.9, 121.8)
- added D1: 1N4934, simple002:DO-41, F.Cu at (112.5, 89.7)
- added D2: 1N4934, simple002:DO-41, F.Cu at (112.5, 93.6)
- added D3: 1N4934, simple002:DO-41, F.Cu at (112.5, 97.5)
- added D4: 1N4934, simple002:DO-41, F.Cu at (112.5, 101.4)
- added D5: 1N4934, simple002:DO-41, F.Cu at (112.5, 105.3)
- added D6: 1N4934, simple002:DO-41, F.Cu at (112.5, 109.2)
- added FAN1: FAN1, simple002:FAN4, F.Cu at (85.7, 75.7)
- added FAN2: FAN2, simple002:FAN4, F.Cu at (85.7, 83.0)
- added FAN3: FAN3, simple002:FAN4, F.Cu at (85.7, 90.3)
- added FAN4: FAN4, simple002:FAN4, F.Cu at (85.7, 97.6)
- added FAN5: FAN5, simple002:FAN4, F.Cu at (85.7, 104.8)
- added FAN6: FAN6, simple002:FAN4, F.Cu at (85.7, 112.1)
- added HDR1: 641737-1, simple002:641737-1, F.Cu at (113.6, 74.8)
- added J1: 1725711, 1725711:1725711, F.Cu at (86.4, 63.5)
- added R1: 10K, simple002:V234_12, F.Cu at (99.0, 90.1)
- added R2: 10K, simple002:V234_12, F.Cu at (99.0, 94.8)
- added R3: 10K, simple002:V234_12, F.Cu at (99.0, 99.5)
- added R4: 10K, simple002:V234_12, F.Cu at (99.0, 104.2)
- added R5: 10K, simple002:V234_12, F.Cu at (99.0, 109.0)
- added R6: JMP, simple002:R0402, F.Cu at (112.1, 112.3)
- added SH1: SHORTT5, simple002:SHORT_TOP-50, F.Cu at (111.8, 114.5)
- added TEENSY0: TEENSY_3.5_DIL+4, simple002:TEENSY_3.5_DIL+4, F.Cu at (70.4, 104.1)
- added TEMP1: TEMP1, simple002:SENSOR2, F.Cu at (94.7, 113.4)
- added TEMP2: TEMP2, simple002:SENSOR2, F.Cu at (94.7, 117.4)
- added TEMP3: TEMP3, simple002:SENSOR2, F.Cu at (94.7, 121.5)
- added TEMP4: TEMP4, simple002:SENSOR2, F.Cu at (94.7, 125.5)
- added TEMP5: TEMP5, simple002:SENSOR2, F.Cu at (94.7, 129.6)
